File: board/SD_Swap/SD_Swap.kicad_sch (KiCad schematic)
At the start: 44 parts, among them J1 USB_C, Q1 Q_Dual_PNP_PNP_E1B1C2E2B2C1, U1 74LVC2G14, U2 RTS5306E, U3 PCB_SD, U4 93AAxxAT, U5 TS3A27518ERTW, U6 SD_SOCKET, U7 AZ1117-3.3, Y1 12MHz

Commit message: Update silkscreen to include logo and revision number
Other:
- title: SD SWAP -> SDWire3
Changed lines of the file:
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@@
 	(paper "A4")
 	(title_block
-		(title "SD SWAP")
-		(date "2023-08-26")
-		(rev "V1.1")
+		(title "SDWire3")
+		(date "2025-01-26")
+		(rev "V1.0")
 	)
 	(junction

Commit message: update part numbers
Parts:
- D2: LCSC C264332 -> C970148
- Q1: LCSC C703623 -> C111730
- R11, R4, R5: LCSC C423334 -> C180341
- R7, R8: LCSC C2991668 -> C106229
- U6: LCSC (none) -> C724031
Changed lines of the file:
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@@
 			)
 		)
-		(property "LCSC" "C423334"
+		(property "LCSC" "C180341"
 			(at 111.76 70.358 0)
 			(effects
@@
 			)
 		)
-		(property "LCSC" "C703623"
+		(property "LCSC" "C111730"
 			(at 95.25 41.148 0)
 			(effects
@@
 			)
 		)
-		(property "LCSC" "C703623"
+		(property "LCSC" "C111730"
 			(at 111.76 41.148 0)
 			(effects
@@
 			)
 		)
-		(property "LCSC" "C423334"
+		(property "LCSC" "C180341"
 			(at 147.574 160.274 0)
 			(effects
@@
 			)
 		)
-		(property "LCSC" "C423334"
+		(property "LCSC" "C180341"
 			(at 116.332 102.108 0)
 			(effects
@@
 			)
 		)
-		(property "LCSC" "C2991668"
+		(property "LCSC" "C106229"
 			(at 95.25 51.562 0)
 			(effects
@@
 			)
 		)
-		(property "LCSC" "~"
+		(property "LCSC" "C724031"
 			(at 239.014 54.102 0)
 			(effects
@@
 			)
 		)
-		(property "LCSC" "C2991668"
+		(property "LCSC" "C106229"
 			(at 111.76 51.562 0)
 			(effects
@@
 			)
 		)
-		(property "LCSC" "C264332"
+		(property "LCSC" "C970148"
 			(at 67.564 93.853 0)
 			(effects
